File: kicad/mdb-vmc-esp32s3.kicad_sch (KiCad schematic)
At the start: 53 parts, among them J1 MDB_Connector, J2 USB_C_Receptacle_USB2.0_16P, J4 Conn_Coaxial, J8 Conn_01x04_Pin, J9 MDB_Connector, Q8 MMBT3904, SW1 SW_Push, U1 TLP785, U3 ESP32-S3FH4R2, U4 TLP785, U5 LM2594HVM-3.3, U7 MT3608, Y1 Crystal_GND24

Commit message: tlp7185^Co tlp785
Parts:
- U1, U4: LCSC# C128776 -> C45445
Changed lines of the file:
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@@
 			)
 		)
-		(property "LCSC#" "C128776"
+		(property "LCSC#" "C45445"
 			(at 358.14 82.55 0)
 			(effects
@@
 			)
 		)
-		(property "LCSC#" "C128776"
+		(property "LCSC#" "C45445"
 			(at 358.14 97.79 0)
 			(effects

Commit message: Add files via upload
Parts:
- added D2, D6: D_Schottky, Diode_SMD:D_SOD-123, symbol Device:D_Schottky
- added J5: Barrel_Jack, Connector_BarrelJack:BarrelJack_Horizontal, symbol Connector:Barrel_Jack
Connections:
- net GND: now also J5.2
- net vin: now also D2.1 (K), D6.1 (K); no longer J1.1 (Pin_1)
- new net: D6.2 (A), J5.1
- new net: D2.2 (A), J1.1 (Pin_1)
