File: kicad/mdb-ai-bridge-esp32s3/mdb-ai-bridge-esp32s3.kicad_sch (KiCad schematic)
At the start: 0 parts

Commit message: refactor(kicad): rename mdb-vmc-esp32s3 to mdb-bridge-esp32s3
Update directory, filenames, and internal .kicad_pro reference.

Co-Authored-By: Claude Sonnet 4.6 <noreply@anthropic.com>
Parts:
- added C1, C15: 1uF, Capacitor_SMD:C_0603_1608Metric, symbol Device:C
- added C12, C14, C16, C17, C7: 0.1uF, Capacitor_SMD:C_0603_1608Metric, symbol Device:C
- added C13: 10uF, Capacitor_SMD:C_0603_1608Metric, symbol Device:C
- added C18, C22: 22pF, Capacitor_SMD:C_0603_1608Metric, symbol Device:C
- added C2: 220uF, Capacitor_Tantalum_SMD:CP_EIA-3528-21_Kemet-B, symbol Device:C_Polarized
- added C3: 100uF, Capacitor_SMD:CP_Elec_6.3x5.8, symbol Device:C_Polarized
- added C4: 1.8pf, Capacitor_SMD:C_0603_1608Metric, symbol Device:C
- added C5, C6: 12pF, Capacitor_SMD:C_0603_1608Metric, symbol Device:C
- added D1, D3, D5: D_Schottky, Diode_SMD:D_SOD-123, symbol Device:D_Schottky
- added D4: XL-2121RGBC-2812B, LED_SMD:LED_WS2812B-2020_PLCC4_2.0x2.0mm, symbol LED:WS2812B-2020
- added FB2: FerriteBead_Small, Inductor_SMD:L_0603_1608Metric, symbol Device:FerriteBead_Small
- added H1: MountingHole, MountingHole:MountingHole_2.1mm, symbol Mechanical:MountingHole
- added J1, J9: MDB_Connector, Connector_Molex:Molex_Mini-Fit_Jr_5566-06A_2x03_P4.20mm_Vertical, symbol Connector_Generic:Conn_02x03_Top_Bottom
- added J2: USB_C_Receptacle_USB2.0_16P, Connector_USB:USB_C_Receptacle_G-Switch_GT-USB-7010ASV, symbol Connector:USB_C_Receptacle_USB2.0_16P
- added J4: Conn_Coaxial, Connector_Coaxial:U.FL_Hirose_U.FL-R-SMT-1_Vertical, symbol Connector:Conn_Coaxial
- added J8: Conn_01x04_Pin, Connector_JST:JST_PH_B4B-PH-K_1x04_P2.00mm_Vertical, symbol Connector:Conn_01x04_Pin
- added L1: 2.4nh, Inductor_SMD:L_0603_1608Metric, symbol Device:L
- added L2: 100uH, Inductor_SMD:L_7.3x7.3_H3.5, symbol Device:L
- added L5: 4.7uF, Inductor_SMD:L_APV_ANR3015, symbol Device:L
- added Q8: MMBT3904, Package_TO_SOT_SMD:SOT-23, symbol Transistor_BJT:MMBT3904
- added R1, R10, R32: 1k, Resistor_SMD:R_0603_1608Metric, symbol Device:R
- added R2, R5: 470ohm, Resistor_SMD:R_0603_1608Metric, symbol Device:R
- added R24, R25, R31: 4K7, Resistor_SMD:R_0603_1608Metric, symbol Device:R
- added R26: 15k, Resistor_SMD:R_0603_1608Metric, symbol Device:R
- added R28: 110k, Resistor_SMD:R_0603_1608Metric, symbol Device:R
- added R3, R4, R6, R9: 10k, Resistor_SMD:R_0603_1608Metric, symbol Device:R
- added R7, R8: 5.1k, Resistor_SMD:R_0603_1608Metric, symbol Device:R
- added SW1: SW_Push, Button_Switch_SMD:SW_Tactile_SPST_NO_Straight_CK_PTS636Sx25SMTRLFS, symbol Switch:SW_Push
- added U1, U4: TLP785, Package_SO:SOP-4_3.8x4.1mm_P2.54mm, symbol Isolator:TLP785
- added U3: ESP32-S3FH4R2, Package_DFN_QFN:QFN-56-1EP_7x7mm_P0.4mm_EP4x4mm, symbol PCM_Espressif:ESP32-S3
- added U5: LM2594HVM-3.3, Package_SO:SOIC-8_3.9x4.9mm_P1.27mm, symbol Regulator_Switching:LM2594HVM-3.3
- added U7: MT3608, Package_TO_SOT_SMD:SOT-23-6, symbol Regulator_Switching:MT3608
- added Y1: Crystal_GND24, Crystal:Crystal_SMD_3225-4Pin_3.2x2.5mm, symbol Device:Crystal_GND24
Connections:
- new net: R2.2, U4.1
- new net: R5.2, U1.1
- new net: D3.2 (A), L5.2, U7.1 (SW)
- new net: D5.2 (A), J2.A4 (VBUS), J2.A9 (VBUS), J2.B4 (VBUS), J2.B9 (VBUS)
- new net: J2.A5 (CC1), R8.1
- new net: J2.B5 (CC2), R7.1
- new net: R26.1, R28.2, U7.3 (FB)
- new net: D1.1 (K), L2.1, U5.8 (OUT)
- new net: C1.1, R3.2, U3.4 (CHIP_PU/RESET)
- new net: C6.2, U3.54 (XTAL_P), Y1.1
- new net: R9.1, U3.52 (GPIO46)
- new net: C5.2, U3.53 (XTAL_N), Y1.3
- new net: R6.1, U3.51 (GPIO45)
- new net: C4.2, U3.1 (LNA_IN/RF)
- new net: Q8.1 (B), R1.1
- new net: C4.1, J4.1 (In), L1.1
- new net +3V3: C12.2, C13.2, C15.2, C16.1, C17.1, C18.2, C2.1, C7.1, D4.2 (VDD), FB2.2, J8.2 (Pin_2), L2.2, L5.1, R10.1, R24.2, R25.2, R3.1, R32.2, R4.2, R5.1, U3.20 (VDD3P3_RTC), U3.46 (VDD3P3_CPU), U3.55 (VDDA), U3.56 (VDDA), U5.4 (FB), U7.4 (EN), U7.5 (IN)
- new net +5V: C22.2, D3.1 (K), R28.1, R31.2
- new net GND: C1.2, C12.1, C13.1, C14.1, C15.1, C16.2, C17.2, C18.1, C2.2, C22.1, C3.2, C5.1, C6.1, C7.2, D1.2 (A), D4.4 (VSS), J1.2 (Pin_2), J2.A1 (GND), J2.A12 (GND), J2.B1 (GND), J2.B12 (GND), J2.S1 (SHIELD), J4.2 (Ext), J8.1 (Pin_1), J9.2 (Pin_2), J9.6 (Pin_6), L1.2, Q8.2 (E), R26.2, R6.2, R7.2, R8.2, R9.2, SW1.2, U3.57 (GND), U4.3, U5.5 (~{ON}/OFF), U5.6 (GND), U7.2 (GND), Y1.2, Y1.4
- new net VDD3P3: C14.2, FB2.1, U3.2 (VDD3P3), U3.3 (VDD3P3)
- new net boot: R4.1, SW1.1, U3.5 (GPIO0/BOOT)
- new net io1: J9.4 (Pin_4), R32.1, U3.6 (GPIO1/ADC1_CH0)
- new net io10: J8.3 (Pin_3), R24.1, U3.15 (GPIO10/ADC1_CH9)
- new net io11: J8.4 (Pin_4), R25.1, U3.16 (GPIO11/ADC2_CH0)
- new net io12: U3.17 (GPIO12/ADC2_CH1)
- new net io13: U3.18 (GPIO13/ADC2_CH2)
- new net io14: U3.19 (GPIO14/ADC2_CH3)
- new net io17: U3.23 (GPIO17/ADC2_CH6)
- new net io18: U3.24 (GPIO18/ADC2_CH7)
- new net io2: R1.2, U3.7 (GPIO2/ADC1_CH1)
- new net io21: D4.1 (DIN), U3.27 (GPIO21)
- new net io4: R10.2, U3.9 (GPIO4/ADC1_CH3), U4.4
- new net io5: U1.2, U3.10 (GPIO5/ADC1_CH4)
- new net io6: U3.11 (GPIO6/ADC1_CH5)
- new net io7: U3.12 (GPIO7/ADC1_CH6)
- new net io8: U3.13 (GPIO8/ADC1_CH7)
- new net io9: U3.14 (GPIO9/ADC1_CH8)
- new net mdb_communications_common: J1.6 (Pin_6), U1.3, U4.2
- new net mdb_controller_transmit: J9.5 (Pin_5), Q8.3 (C), R31.1
- new net mdb_master_receive: J1.4 (Pin_4), U1.4
- new net mdb_master_transmit: J1.5 (Pin_5), R2.1
- new net u0rxd: U3.50 (U0RXD/PROG/GPIO44)
- new net u0txd: U3.49 (U0TXD/PROG/GPIO43)
- new net usb+: J2.A6 (D+), J2.B6 (D+), U3.26 (GPIO20/USB_D+/ADC2_CH9)
- new net usb-: J2.A7 (D-), J2.B7 (D-), U3.25 (GPIO19/USB_D-/ADC2_CH8)
- new net vin: C3.1, D5.1 (K), J1.1 (Pin_1), J9.1 (Pin_1), U5.7 (VIN)
- no-connect marks 0 -> 31

Commit message: feat(kicad): update mdb-ai-bridge-esp32s3 schematic
Co-Authored-By: Claude Sonnet 4.6 <noreply@anthropic.com>
Parts:
- removed C12, C14, C16, C17, C7: 0.1uF, Capacitor_SMD:C_0603_1608Metric, symbol Device:C
- removed C13: 10uF, Capacitor_SMD:C_0603_1608Metric, symbol Device:C
- removed C15: 1uF, Capacitor_SMD:C_0603_1608Metric, symbol Device:C
- removed C18, C22: 22pF, Capacitor_SMD:C_0603_1608Metric, symbol Device:C
- removed C2: 220uF, Capacitor_Tantalum_SMD:CP_EIA-3528-21_Kemet-B, symbol Device:C_Polarized
- removed C3: 100uF, Capacitor_SMD:CP_Elec_6.3x5.8, symbol Device:C_Polarized
- removed C4: 1.8pf, Capacitor_SMD:C_0603_1608Metric, symbol Device:C
- removed C5, C6: 12pF, Capacitor_SMD:C_0603_1608Metric, symbol Device:C
- removed D1, D3, D5: D_Schottky, Diode_SMD:D_SOD-123, symbol Device:D_Schottky
- removed D4: XL-2121RGBC-2812B, LED_SMD:LED_WS2812B-2020_PLCC4_2.0x2.0mm, symbol LED:WS2812B-2020
- removed FB2: FerriteBead_Small, Inductor_SMD:L_0603_1608Metric, symbol Device:FerriteBead_Small
- removed H1: MountingHole, MountingHole:MountingHole_2.1mm, symbol Mechanical:MountingHole
- removed J1, J9: MDB_Connector, Connector_Molex:Molex_Mini-Fit_Jr_5566-06A_2x03_P4.20mm_Vertical, symbol Connector_Generic:Conn_02x03_Top_Bottom
- removed J2: USB_C_Receptacle_USB2.0_16P, Connector_USB:USB_C_Receptacle_G-Switch_GT-USB-7010ASV, symbol Connector:USB_C_Receptacle_USB2.0_16P
- removed J4: Conn_Coaxial, Connector_Coaxial:U.FL_Hirose_U.FL-R-SMT-1_Vertical, symbol Connector:Conn_Coaxial
- removed J8: Conn_01x04_Pin, Connector_JST:JST_PH_B4B-PH-K_1x04_P2.00mm_Vertical, symbol Connector:Conn_01x04_Pin
- removed L1: 2.4nh, Inductor_SMD:L_0603_1608Metric, symbol Device:L
- removed L2: 100uH, Inductor_SMD:L_7.3x7.3_H3.5, symbol Device:L
- removed L5: 4.7uF, Inductor_SMD:L_APV_ANR3015, symbol Device:L
- removed Q8: MMBT3904, Package_TO_SOT_SMD:SOT-23, symbol Transistor_BJT:MMBT3904
- removed R10, R32: 1k, Resistor_SMD:R_0603_1608Metric, symbol Device:R
- removed R24, R25, R31: 4K7, Resistor_SMD:R_0603_1608Metric, symbol Device:R
- removed R26: 15k, Resistor_SMD:R_0603_1608Metric, symbol Device:R
- removed R28: 110k, Resistor_SMD:R_0603_1608Metric, symbol Device:R
- removed SW1: SW_Push, Button_Switch_SMD:SW_Tactile_SPST_NO_Straight_CK_PTS636Sx25SMTRLFS, symbol Switch:SW_Push
- removed U1, U4: TLP785, Package_SO:SOP-4_3.8x4.1mm_P2.54mm, symbol Isolator:TLP785
- removed U3: ESP32-S3FH4R2, Package_DFN_QFN:QFN-56-1EP_7x7mm_P0.4mm_EP4x4mm, symbol PCM_Espressif:ESP32-S3
- removed U5: LM2594HVM-3.3, Package_SO:SOIC-8_3.9x4.9mm_P1.27mm, symbol Regulator_Switching:LM2594HVM-3.3
- removed U7: MT3608, Package_TO_SOT_SMD:SOT-23-6, symbol Regulator_Switching:MT3608
- removed Y1: Crystal_GND24, Crystal:Crystal_SMD_3225-4Pin_3.2x2.5mm, symbol Device:Crystal_GND24
- added AE3: Antenna, RF_Antenna:Texas_SWRA117D_2.4GHz_Left, symbol Device:Antenna
- added C10, C29, C37, C43, C44, C45, C46, C48, C49, C52, C53, C56, C57, C9: 0.1uF, Capacitor_SMD:C_0603_1608Metric, symbol Device:C
- added C11, C20, C31, C32, C35, C36, C39, C40: 12pF, Capacitor_SMD:C_0603_1608Metric, symbol Device:C
- added C19, C42, C50, C54: 10uF, Capacitor_SMD:C_0603_1608Metric, symbol Device:C
- added C30, C34, C38, C47, C51, C55, C8: 1uF, Capacitor_SMD:C_0603_1608Metric, symbol Device:C
- added C33: 1.8pf, Capacitor_SMD:C_0603_1608Metric, symbol Device:C
- added C41: 22uF, Capacitor_SMD:C_0603_1608Metric, symbol Device:C
- added D10, D11, D9: XL-2121RGBC-2812B, LED_SMD:LED_WS2812B-2020_PLCC4_2.0x2.0mm, symbol LED:WS2812B-2020
- added D8: D_Schottky, Diode_SMD:D_SOD-123, symbol Device:D_Schottky
- added FB3, FB4, FB5: FerriteBead_Small, Inductor_SMD:L_0603_1608Metric, symbol Device:FerriteBead_Small
- added H2: MountingHole, MountingHole:MountingHole_2.1mm, symbol Mechanical:MountingHole
- added J7: USB_C_Receptacle_USB2.0_16P, Connector_USB:USB_C_Receptacle_G-Switch_GT-USB-7010ASV, symbol Connector:USB_C_Receptacle_USB2.0_16P
- added L7: 2.4nh, Inductor_SMD:L_0603_1608Metric, symbol Device:L
- added R11: 12k, Resistor_SMD:R_0603_1608Metric, symbol Device:R
- added R23, R27, R29, R30, R33, R34, R35, R36, R37, R38, R39, R40, R43: 10k, Resistor_SMD:R_0603_1608Metric, symbol Device:R
- added R41, R42: 5.1k, Resistor_SMD:R_0603_1608Metric, symbol Device:R
- added R44, R45: 4K7, Resistor_SMD:R_0603_1608Metric, symbol Device:R
- added SW3, SW4, SW5, SW6, SW7, SW8, SW9: SW_Push, Button_Switch_SMD:SW_Tactile_SPST_NO_Straight_CK_PTS636Sx25SMTRLFS, symbol Switch:SW_Push
- added U10, U11, U12: ESP32-S3FH4R2, Package_DFN_QFN:QFN-56-1EP_7x7mm_P0.4mm_EP4x4mm, symbol PCM_Espressif:ESP32-S3
- added U13: AMS1117-3.3, Package_TO_SOT_SMD:SOT-223-3_TabPin2, symbol Regulator_Linear:AMS1117-3.3
- added U14: USB2514B_Bi, Package_DFN_QFN:QFN-36-1EP_6x6mm_P0.5mm_EP3.7x3.7mm, symbol Interface_USB:USB2514B_Bi
- added Y2, Y3, Y4, Y5: Crystal_GND24, Crystal:Crystal_SMD_3225-4Pin_3.2x2.5mm, symbol Device:Crystal_GND24
- R1: value 1k -> 10k; LCSC# C2907113 -> C98220
- R2, R5: value 470ohm -> 100k; LCSC# C114669 -> (none)
- R3, R4, R6: value 10k -> 100k; LCSC# C98220 -> (none)
- R7: value 5.1k -> 100k; LCSC# C394543 -> (none)
- R8: value 5.1k -> 10k; LCSC# C394543 -> C98220
Connections:
- net boot is gone; now on net GND: R4.1
- net +3V3: now also R1.1, R8.2, R9.2, C10.1, C19.2, C29.2, C41.2, C43.2, C44.2, C47.2, C48.1, C49.1, C50.2, C51.2, C52.1, C53.1, C54.2, C55.2, C56.1, C57.1, C8.2, C9.1, D10.2 (VDD), D11.2 (VDD), D9.2 (VDD), FB3.2, FB4.2, FB5.2, R23.1, R29.2, R33.1, R35.2, R37.1, R39.2, R43.2, R44.2, R45.2, U10.20 (VDD3P3_RTC), U10.46 (VDD3P3_CPU), U10.55 (VDDA), U10.56 (VDDA), U11.20 (VDD3P3_RTC), U11.46 (VDD3P3_CPU), U11.55 (VDDA), U11.56 (VDDA), U12.20 (VDD3P3_RTC), U12.46 (VDD3P3_CPU), U12.55 (VDDA), U12.56 (VDDA), U13.2 (VO), U14.10 (VDDA33), U14.15 (VDD33), U14.23 (VDD33), U14.29 (VDDA33), U14.36 (VDDA33), U14.5 (VDDA33); no longer R3.1, R4.2
- net GND: now also R2.1, R3.1, C10.2, C11.1, C19.1, C20.1, C29.1, C30.2, C31.1, C32.1, C34.2, C35.1, C36.1, C37.1, C38.2, C39.1, C40.1, C41.1, C42.1, C43.1, C44.1, C45.1, C46.1, C47.1, C48.2, C49.2, C50.1, C51.1, C52.2, C53.2, C54.1, C55.1, C56.2, C57.2, C8.1, C9.2, D10.4 (VSS), D11.4 (VSS), D9.4 (VSS), J7.A1 (GND), J7.A12 (GND), J7.B1 (GND), J7.B12 (GND), J7.S1 (SHIELD), L7.2, R11.1, R27.2, R30.2, R34.2, R36.2, R38.2, R40.2, R41.2, R42.2, SW3.2, SW4.2, SW5.2, SW6.2, SW7.2, SW8.2, SW9.2, U10.57 (GND), U11.57 (GND), U12.57 (GND), U13.1 (GND), U14.37 (VSS), Y2.2, Y2.4, Y3.2, Y3.4, Y4.2, Y4.4, Y5.2, Y5.4; no longer R7.2, R8.2, R9.2
- net VDD3P3: now also C37.2, C45.2, C46.2, FB3.1, FB4.1, FB5.1, U10.2 (VDD3P3), U10.3 (VDD3P3), U11.2 (VDD3P3), U11.3 (VDD3P3), U12.2 (VDD3P3), U12.3 (VDD3P3)
- net io10: now also R45.1, U10.15 (GPIO10/ADC1_CH9), U11.15 (GPIO10/ADC1_CH9), U12.15 (GPIO10/ADC1_CH9)
- net io11: now also R44.1, U10.16 (GPIO11/ADC2_CH0), U11.16 (GPIO11/ADC2_CH0), U12.16 (GPIO11/ADC2_CH0)
- net mdb_controller_transmit: now also U10.9 (GPIO4/ADC1_CH3), U11.7 (GPIO2/ADC1_CH1)
- net mdb_master_receive: now also U11.10 (GPIO5/ADC1_CH4), U12.6 (GPIO1/ADC1_CH0)
- net mdb_master_transmit: now also U11.9 (GPIO4/ADC1_CH3), U12.7 (GPIO2/ADC1_CH1); no longer R2.1
- net u0rxd: now also U11.14 (GPIO9/ADC1_CH8), U12.50 (U0RXD/PROG/GPIO44)
- net u0txd: now also U11.13 (GPIO8/ADC1_CH7), U12.49 (U0TXD/PROG/GPIO43)
- net usb+: now also J7.A6 (D+), J7.B6 (D+), U14.31 (USBDP_UP)
- net usb-: now also J7.A7 (D-), J7.B7 (D-), U14.30 (USBDM_UP)
- net vin: now also C42.2, D8.1 (K), U13.3 (VI)
- net at R2.2: now also U14.24 (SCL/SMBCLK/CFG_SEL0)
- net at R5.2: now also U14.25 (HS_IND/CFG_SEL1)
- net at R8.1: now also U14.8 (USBDM_DN4/PRT_DIS_M4)
- net at R7.1: now also D8.2 (A), J7.A4 (VBUS), J7.A9 (VBUS), J7.B4 (VBUS), J7.B9 (VBUS)
- net at R3.2: now also U14.22 (SDA/SMBDATA/NON_REM1); no longer C1.1
- net at R9.1: now also U14.9 (USBDP_DN4/PRT_DIS_P4)
- net vbus_det: now reaches R6.1
- net vbus_det: now also R7.2, U14.27 (VBUS_DET)
- net io2: no longer names the net of R1.2
- net io2: now also C1.1, U14.26 (RESET_N)
- new net: C30.1, R23.2, SW7.1, U10.4 (CHIP_PU/RESET)
- new net: R30.1, U10.51 (GPIO45)
- new net: R4.2, U14.28 (SUSP_IND/LOCAL_PWR/NON_REM0)
- new net: C20.2, U14.32 (XTALOUT), Y2.1
- new net: C11.2, U14.33 (XTALIN/CLKIN), Y2.3
- new net: R11.2, U14.35 (RBIAS)
- new net: C40.2, U12.54 (XTAL_P), Y5.1
- new net: C39.2, U12.53 (XTAL_N), Y5.3
- new net: R36.1, U11.51 (GPIO45)
- new net: C38.1, R37.2, SW6.1, U12.4 (CHIP_PU/RESET)
- new net: C34.1, R33.2, SW8.1, U11.4 (CHIP_PU/RESET)
- new net: D11.1 (DIN), U10.27 (GPIO21)
- new net: R29.1, SW3.1, U10.5 (GPIO0/BOOT)
- new net: R27.1, U10.52 (GPIO46)
- new net: C31.2, U10.53 (XTAL_N), Y3.3
- new net: C32.2, U10.54 (XTAL_P), Y3.1
- new net: R43.1, SW9.1, U10.6 (GPIO1/ADC1_CH0)
- new net: J7.A5 (CC1), R42.1
- new net: J7.B5 (CC2), R41.1
- new net: R35.1, SW4.1, U11.5 (GPIO0/BOOT)
- new net: R40.1, U12.51 (GPIO45)
- new net: C35.2, U11.53 (XTAL_N), Y4.3
- new net: R34.1, U11.52 (GPIO46)
- new net: AE3.1 (A), C33.1, L7.1
- new net: C33.2, U11.1 (LNA_IN/RF)
- new net: D9.1 (DIN), U11.27 (GPIO21)
- new net: D10.1 (DIN), U12.27 (GPIO21)
- new net: R39.1, SW5.1, U12.5 (GPIO0/BOOT)
- new net: R38.1, U12.52 (GPIO46)
- new net: C36.2, U11.54 (XTAL_P), Y4.1
- new net mdb_controller_receive: U10.10 (GPIO5/ADC1_CH4), U11.6 (GPIO1/ADC1_CH0)
- new net usb+_1: U10.26 (GPIO20/USB_D+/ADC2_CH9), U14.2 (USBDP_DN1/PRT_DIS_P1)
- new net usb+_2: U11.26 (GPIO20/USB_D+/ADC2_CH9), U14.4 (USBDP_DN2/PRT_DIS_P2)
- new net usb+_3: U12.26 (GPIO20/USB_D+/ADC2_CH9), U14.7 (USBDP_DN3/PRT_DIS_P3)
- new net usb-_1: U10.25 (GPIO19/USB_D-/ADC2_CH8), U14.1 (USBDM_DN1/PRT_DIS_M1)
- new net usb-_2: U11.25 (GPIO19/USB_D-/ADC2_CH8), U14.3 (USBDM_DN2/PRT_DIS_M2)
- new net usb-_3: U12.25 (GPIO19/USB_D-/ADC2_CH8), U14.6 (USBDM_DN3/PRT_DIS_M3)
- no-connect marks 31 -> 76
Other:
- note added: "0.1 µF on VDD33 and 1 µF + 0.1 µF on the analog supply;"

Commit message: feat(kicad): fill missing LCSC# for 9 components in mdb-ai-bridge
Co-Authored-By: Claude Sonnet 4.6 <noreply@anthropic.com>
Parts:
- C41: LCSC# (none) -> C15500
- C42: LCSC# (none) -> C6119864
- R11: LCSC# (none) -> C22790
- R2, R3, R4, R5, R6, R7: LCSC# (none) -> C25803
Changed lines of the file:
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@@
 			)
 		)
-		(property "LCSC#" ""
+		(property "LCSC#" "C15500"
 			(at 400.05 347.98 90)
 			(effects
@@
 			)
 		)
-		(property "LCSC#" ""
+		(property "LCSC#" "C25803"
 			(at 316.23 326.39 90)
 			(effects
@@
 			)
 		)
-		(property "LCSC#" ""
+		(property "LCSC#" "C25803"
 			(at 309.88 87.63 90)
 			(effects
@@
 			)
 		)
-		(property "LCSC#" ""
+		(property "LCSC#" "C25803"
 			(at 314.96 95.25 90)
 			(effects
@@
 			)
 		)
-		(property "LCSC#" ""
+		(property "LCSC#" "C6119864"
 			(at 372.11 346.71 90)
 			(effects
@@
 			)
 		)
-		(property "LCSC#" ""
+		(property "LCSC#" "C22790"
 			(at 307.34 64.77 90)
 			(effects
@@
 			)
 		)
-		(property "LCSC#" ""
+		(property "LCSC#" "C25803"
 			(at 292.1 92.71 90)
 			(effects
@@
 			)
 		)
-		(property "LCSC#" ""
+		(property "LCSC#" "C25803"
 			(at 327.66 326.39 90)
 			(effects
@@
 			)
 		)
-		(property "LCSC#" ""
+		(property "LCSC#" "C25803"
 			(at 300.99 90.17 90)
 			(effects

Commit message: feat(kicad): add LCSC# field to remaining 4 components
U13 (AMS1117-3.3) -> C6186, U14 (USB2514B_Bi) -> C510949.
AE3 and H2 get empty field (PCB antenna / mechanical hole).

Co-Authored-By: Claude Sonnet 4.6 <noreply@anthropic.com>
Parts:
- U13: LCSC# (none) -> C6186
- U14: LCSC# (none) -> C510949
Changed lines of the file:
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@@
 			)
 		)
+		(property "LCSC#" "C510949"
+			(at 0 0 0)
+			(effects
+				(font
+					(size 1.27 1.27)
+				)
+				(hide yes)
+			)
+		)
 		(property "Datasheet" "http://ww1.microchip.com/downloads/en/DeviceDoc/00001692C.pdf"
 			(at 391.16 107.95 0)
@@
 			)
 		)
+		(property "LCSC#" "C6186"
+			(at 0 0 0)
+			(effects
+				(font
+					(size 1.27 1.27)
+				)
+				(hide yes)
+			)
+		)
 		(property "Datasheet" "http://www.advanced-monolithic.com/pdf/ds1117.pdf"
 			(at 386.08 347.98 0)
@@
 			)
 		)
+		(property "LCSC#" ""
+			(at 0 0 0)
+			(effects
+				(font
+					(size 1.27 1.27)
+				)
+				(hide yes)
+			)
+		)
 		(property "Datasheet" "~"
 			(at 560.07 34.29 0)
@@
 			(effects
 				(font
+					(size 1.27 1.27)
+				)
+				(hide yes)
+			)
+		)
+		(property "LCSC#" ""
+			(at 0 0 0)
+			(effects
+				(font

Commit message: feat(kicad): add PCB layout and update schematic for mdb-ai-bridge-esp32s3
PCB was previously a placeholder (empty board). Full routing and component
placement now added. Schematic also updated with matching changes.

Co-Authored-By: Claude Sonnet 4.6 <noreply@anthropic.com>
Parts:
- added C2: 0.1uF, Capacitor_SMD:C_0603_1608Metric, symbol Device:C
- added J2: Conn_02x08_Top_Bottom, Connector_PinHeader_2.54mm:PinHeader_2x08_P2.54mm_Vertical, symbol Connector_Generic:Conn_02x08_Top_Bottom
Connections:
- net +3V3: now also C2.1, J2.1 (Pin_1)
- net GND: now also C2.2, J2.11 (Pin_11), J2.12 (Pin_12), J2.2 (Pin_2), J2.3 (Pin_3), J2.7 (Pin_7), J2.8 (Pin_8)
- net io10: now also J2.9 (Pin_9)
- net io11: now also J2.10 (Pin_10)
- net mdb_controller_receive: now also J2.6 (Pin_6)
- net mdb_controller_transmit: now also J2.5 (Pin_5)
- net vin: now also J2.4 (Pin_4)
- net io12: now reaches U11.17 (GPIO12/ADC2_CH1)
- net io12: now also J2.13 (Pin_13)
- net io13: now reaches U11.18 (GPIO13/ADC2_CH2)
- net io13: now also J2.14 (Pin_14)
- net io14: now reaches U11.19 (GPIO14/ADC2_CH3)
- net io14: now also J2.15 (Pin_15)
- net io17: now reaches U11.23 (GPIO17/ADC2_CH6)
- net io17: now also J2.16 (Pin_16)
