File: kicad/mdb-ai-bridge-esp32s3/mdb-ai-bridge-esp32s3.kicad_sch (KiCad schematic)
At the start: 92 parts, among them J2 Conn_02x08_Top_Bottom, J7 USB_C_Receptacle_USB2.0_16P, SW3 SW_Push, SW4 SW_Push, SW5 SW_Push, SW6 SW_Push, SW7 SW_Push, SW8 SW_Push, SW9 SW_Push, U10 ESP32-S3FH4R2, U11 ESP32-S3FH4R2, U12 ESP32-S3FH4R2, U13 AMS1117-3.3, U14 USB2514B_Bi, Y2 Crystal_GND24, Y3 Crystal_GND24, Y4 Crystal_GND24, Y5 Crystal_GND24

Commit message: routing...
Parts:
- removed C2: 0.1uF, Capacitor_SMD:C_0603_1608Metric, symbol Device:C
- removed D8: D_Schottky, Diode_SMD:D_SOD-123, symbol Device:D_Schottky
- removed J2: Conn_02x08_Top_Bottom, Connector_PinHeader_2.54mm:PinHeader_2x08_P2.54mm_Vertical, symbol Connector_Generic:Conn_02x08_Top_Bottom
- added C4: 0.1uF, Capacitor_SMD:C_0603_1608Metric, symbol Device:C
- added J3: Conn_02x08_Top_Bottom, Connector_PinHeader_2.54mm:PinHeader_2x08_P2.54mm_Vertical, symbol Connector_Generic:Conn_02x08_Top_Bottom
Connections:
- net vin is gone; now on net +5V: C42.2, U13.3 (VI)
- net +3V3: now also C4.1, J3.1 (Pin_1)
- net GND: now also C4.2, J3.16 (Pin_16), J3.8 (Pin_8), J3.9 (Pin_9)
- net io10: now also J3.2 (Pin_2)
- net io11: now also J3.10 (Pin_10)
- net io12: now also J3.5 (Pin_5)
- net io13: now also J3.13 (Pin_13)
- net io14: now also J3.6 (Pin_6)
- net io17: now also J3.14 (Pin_14)
- net mdb_controller_receive: now also J3.3 (Pin_3)
- net mdb_controller_transmit: now also J3.11 (Pin_11)
- net mdb_master_receive: now also J3.4 (Pin_4)
- net mdb_master_transmit: now also J3.12 (Pin_12)
- net +5V: now reaches J7.A4 (VBUS), J7.A9 (VBUS), J7.B4 (VBUS), J7.B9 (VBUS), R7.1
- net +5V: now also J3.7 (Pin_7)
- net io18: now reaches U11.24 (GPIO18/ADC2_CH7)
- net io18: now also J3.15 (Pin_15)

Commit message: routing...
Parts:
- removed R2, R3: 100k, Resistor_SMD:R_0603_1608Metric, symbol Device:R
Connections:
- net io10: now also U14.22 (SDA/SMBDATA/NON_REM1)
- net io11: now also U14.24 (SCL/SMBCLK/CFG_SEL0)
Changed lines of the file:
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@@
 	)
 	(junction
-		(at 285.75 90.17)
-		(diameter 0)
-		(color 0 0 0 0)
-	)
-	(junction
 		(at 392.43 238.76)
 		(diameter 0)
@@
 	)
 	(junction
-		(at 285.75 92.71)
-		(diameter 0)
-		(color 0 0 0 0)
-	)
-	(junction
 		(at 542.29 222.25)
 		(diameter 0)
@@
 	(wire
 		(pts
-			(xy 306.07 87.63) (xy 285.75 87.63)
-		)
-		(stroke
-			(width 0)
-			(type default)
-		)
-	)
-	(wire
-		(pts
 			(xy 295.91 92.71) (xy 322.58 92.71)
 		)
@@
 	(wire
 		(pts
-			(xy 304.8 90.17) (xy 322.58 90.17)
-		)
-		(stroke
-			(width 0)
-			(type default)
-		)
-	)
-	(wire
-		(pts
 			(xy 421.64 43.18) (xy 434.34 43.18)
 		)
@@
 	(wire
 		(pts
-			(xy 285.75 90.17) (xy 297.18 90.17)
-		)
-		(stroke
-			(width 0)
-			(type default)
-		)
-	)
-	(wire
-		(pts
 			(xy 232.41 335.28) (xy 231.14 335.28)
 		)
@@
 	(wire
 		(pts
-			(xy 313.69 87.63) (xy 322.58 87.63)
-		)
-		(stroke
-			(width 0)
-			(type default)
-		)
-	)
-	(wire
-		(pts
 			(xy 420.37 251.46) (xy 420.37 248.92)
 		)
@@
 	(wire
 		(pts
-			(xy 285.75 92.71) (xy 288.29 92.71)
-		)
-		(stroke
-			(width 0)
-			(type default)
-		)
-	)
-	(wire
-		(pts
 			(xy 165.1 294.64) (xy 168.91 294.64)
 		)
@@
 	(wire
 		(pts
-			(xy 284.48 92.71) (xy 285.75 92.71)
+			(xy 284.48 92.71) (xy 288.29 92.71)
 		)
 		(stroke
@@
 	(wire
 		(pts
-			(xy 285.75 87.63) (xy 285.75 90.17)
-		)
-		(stroke
-			(width 0)
-			(type default)
-		)
-	)
-	(wire
-		(pts
 			(xy 137.16 63.5) (xy 139.7 63.5)
 		)
@@
 	(wire
 		(pts
+			(xy 306.07 90.17) (xy 322.58 90.17)
+		)
+		(stroke
+			(width 0)
+			(type default)
+		)
+	)
+	(wire
+		(pts
 			(xy 217.17 355.6) (xy 217.17 353.06)
 		)
@@
 	(wire
 		(pts
-			(xy 285.75 90.17) (xy 285.75 92.71)
+			(xy 59.69 149.86) (xy 66.04 149.86)
 		)
 		(stroke
@@
 	(wire
 		(pts
-			(xy 59.69 149.86) (xy 66.04 149.86)
+			(xy 54.61 377.19) (xy 54.61 374.65)
 		)
 		(stroke
@@
 	(wire
 		(pts
-			(xy 54.61 377.19) (xy 54.61 374.65)
+			(xy 306.07 87.63) (xy 322.58 87.63)
 		)
 		(stroke
@@
 		)
 	)
+	(label "io11"
+		(at 306.07 87.63 180)
+		(effects
+			(font
+				(size 1.27 1.27)
+			)
+			(justify right bottom)
+		)
+	)
 	(label "usb-_3"
 		(at 382.27 69.85 0)
@@
 		)
 	)
+	(label "io10"
+		(at 306.07 90.17 180)
+		(effects
+			(font
+				(size 1.27 1.27)
+			)
+			(justify right bottom)
+		)
+	)
 	(label "io13"
 		(at 505.46 222.25 0)
@@
 	)
 	(symbol
-		(lib_id "Device:R")
-		(at 309.88 87.63 90)
-		(unit 1)
-		(exclude_from_sim no)
-		(in_bom yes)
-		(on_board yes)
-		(dnp no)
-		(property "Reference" "R2"
-			(at 309.88 81.28 90)
-			(effects
-				(font
-					(size 1.27 1.27)
-				)
-			)
-		)
-		(property "Value" "100k"
-			(at 309.88 83.82 90)
-			(effects
-				(font
-					(size 1.27 1.27)
-				)
-			)
-		)
-		(property "Footprint" "Resistor_SMD:R_0603_1608Metric"
-			(at 309.88 89.408 90)
-			(effects
-				(font
-					(size 1.27 1.27)
-				)
-				(hide yes)
-			)
-		)
-		(property "Datasheet" "~"
-			(at 309.88 87.63 0)
-			(effects
-				(font
-					(size 1.27 1.27)
-				)
-				(hide yes)
-			)
-		)
-		(property "Description" ""
-			(at 309.88 87.63 0)
-			(effects
-				(font
-					(size 1.27 1.27)
-				)
-				(hide yes)
-			)
-		)
-		(property "LCSC#" "C25803"
-			(at 309.88 87.63 90)
-			(effects
-				(font
-					(size 1.27 1.27)
-				)
-				(hide yes)
-			)
-		)
-		(pin "1"
-		)
-		(pin "2"
-		)
-		(instances
-			(project "mdb-ai-bridge-esp32s3"
-				(path "/51cbea2e-46d2-4ff4-a8d6-333c056656c8"
-					(reference "R2")
-					(unit 1)
-				)
-			)
-		)
-	)
-	(symbol
 		(lib_id "power:GND")
 		(at 557.53 222.25 90)
@@
 					(unit 1)
 				)
-			)
-		)
-	)
-	(symbol
-		(lib_id "Device:R")
-		(at 300.99 90.17 90)
-		(unit 1)
-		(exclude_from_sim no)
-		(in_bom yes)
-		(on_board yes)
-		(dnp no)
-		(property "Reference" "R3"
-			(at 300.99 83.82 90)
-			(effects
-				(font
-					(size 1.27 1.27)
-				)
-			)
-		)
-		(property "Value" "100k"
-			(at 300.99 86.36 90)
-			(effects
-				(font
-					(size 1.27 1.27)
-				)
-			)
-		)
-		(property "Footprint" "Resistor_SMD:R_0603_1608Metric"
-			(at 300.99 91.948 90)
-			(effects
-				(font
-					(size 1.27 1.27)
-				)
-				(hide yes)
-			)
-		)
-		(property "Datasheet" "~"
-			(at 300.99 90.17 0)
-			(effects
-				(font
-					(size 1.27 1.27)
-				)
-				(hide yes)
-			)
-		)
-		(property "Description" ""
-			(at 300.99 90.17 0)
-			(effects
-				(font
-					(size 1.27 1.27)
-				)
-				(hide yes)
-			)
-		)
-		(property "LCSC#" "C25803"
-			(at 300.99 90.17 90)
-			(effects
-				(font
-					(size 1.27 1.27)
-				)
-				(hide yes)
-			)
-		)
-		(pin "1"
-		)
-		(pin "2"
-		)
-		(instances
-			(project "mdb-ai-bridge-esp32s3"
-				(path "/51cbea2e-46d2-4ff4-a8d6-333c056656c8"
-					(reference "R3")
-					(unit 1)
-				)

Commit message: routing
Parts:
- added C2, C3: 1uF, Capacitor_SMD:C_0603_1608Metric, symbol Device:C
- added R10, R2, R3: 10k, Resistor_SMD:R_0603_1608Metric, symbol Device:R
- R8, R9: value 10k -> 100k; LCSC# C98220 -> C25803
Connections:
- net +3V3: now also U14.13 (OCS_N1), U14.17 (OCS_N2), U14.19 (OCS_N3), U14.21 (OCS_N4); no longer R5.1, R8.2, R9.2
- net GND: now also R5.1, R8.1, R9.1, C2.1, C3.1, R10.2, R2.2, R3.2
- net io10: no longer U14.22 (SDA/SMBDATA/NON_REM1)
- net io11: no longer U14.24 (SCL/SMBCLK/CFG_SEL0)
- net at U14.12 (PRTPWR1/BC_EN1): now also R2.1
- net at U14.14 (CRFILT): now also C2.2
- net at U14.16 (PRTPWR2/BC_EN2): now also R3.1
- net at U14.18 (PRTPWR3/BC_EN3): now also R10.1
- net at U14.34 (PLLFILT): now also C3.2
- net at U14.8 (USBDM_DN4/PRT_DIS_M4): no longer R8.1
- net at U14.9 (USBDP_DN4/PRT_DIS_P4): no longer R9.1
- new net: R9.2, U14.22 (SDA/SMBDATA/NON_REM1)
- new net: R8.2, U14.24 (SCL/SMBCLK/CFG_SEL0)
- no-connect marks 76 -> 79
