File: kicad/mdb-ai-bridge-esp32s3/mdb-ai-bridge-esp32s3.kicad_sch (KiCad schematic)
At the start: 94 parts, among them J3 Conn_02x08_Top_Bottom, J7 USB_C_Receptacle_USB2.0_16P, SW3 SW_Push, SW4 SW_Push, SW5 SW_Push, SW6 SW_Push, SW7 SW_Push, SW8 SW_Push, SW9 SW_Push, U10 ESP32-S3FH4R2, U11 ESP32-S3FH4R2, U12 ESP32-S3FH4R2, U13 AMS1117-3.3, U14 USB2514B_Bi, Y2 Crystal_GND24, Y3 Crystal_GND24, Y4 Crystal_GND24, Y5 Crystal_GND24

Commit message: fix(hardware): standardize Value field notation in schematics
4K7→4.7k, 470ohm→470R, 1.8pf→1.8pF, 2.4nh→2.4nH,
Crystal_GND24→40MHz/24MHz (por LCSC), FerriteBead_Small→FerriteBead

Co-Authored-By: Claude Sonnet 4.6 <noreply@anthropic.com>
Parts:
- C33: value 1.8pf -> 1.8pF
- FB3, FB4, FB5: value FerriteBead_Small -> FerriteBead
- L7: value 2.4nh -> 2.4nH
- R44, R45: value 4K7 -> 4.7k
- Y2: value Crystal_GND24 -> 24MHz
- Y3, Y4, Y5: value Crystal_GND24 -> 40MHz
Changed lines of the file:
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@@
 			)
 		)
-		(property "Value" "Crystal_GND24"
+		(property "Value" "40MHz"
 			(at 93.98 307.4668 90)
 			(effects
@@
 			)
 		)
-		(property "Value" "Crystal_GND24"
+		(property "Value" "24MHz"
 			(at 295.91 72.5168 90)
 			(effects
@@
 			)
 		)
-		(property "Value" "FerriteBead_Small"
+		(property "Value" "FerriteBead"
 			(at 468.5919 140.97 90)
 			(effects
@@
 			)
 		)
-		(property "Value" "FerriteBead_Small"
+		(property "Value" "FerriteBead"
 			(at 138.3919 39.37 90)
 			(effects
@@
 			)
 		)
-		(property "Value" "4K7"
+		(property "Value" "4.7k"
 			(at 455.93 335.2799 0)
 			(effects
@@
 			)
 		)
-		(property "Value" "2.4nh"
+		(property "Value" "2.4nH"
 			(at 375.92 181.61 0)
 			(effects
@@
 			)
 		)
-		(property "Value" "1.8pf"
+		(property "Value" "1.8pF"
 			(at 381 168.91 90)
 			(effects
@@
 			)
 		)
-		(property "Value" "4K7"
+		(property "Value" "4.7k"
 			(at 464.82 335.2799 0)
 			(effects
@@
 			)
 		)
-		(property "Value" "Crystal_GND24"
+		(property "Value" "40MHz"
 			(at 431.8 194.4368 90)
 			(effects
@@
 			)
 		)
-		(property "Value" "FerriteBead_Small"
+		(property "Value" "FerriteBead"
 			(at 130.7719 254 90)
 			(effects
@@
 			)
 		)
-		(property "Value" "Crystal_GND24"
+		(property "Value" "40MHz"
 			(at 101.6 92.8368 90)
 			(effects
