File: kicad/mdb-ai-bridge-esp32s3/mdb-ai-bridge-esp32s3.kicad_sch (KiCad schematic)
At the start: 94 parts, among them J3 Conn_02x08_Top_Bottom, J7 USB_C_Receptacle_USB2.0_16P, SW3 SW_Push, SW4 SW_Push, SW5 SW_Push, SW6 SW_Push, SW7 SW_Push, SW8 SW_Push, SW9 SW_Push, U10 ESP32-S3FH4R2, U11 ESP32-S3FH4R2, U12 ESP32-S3FH4R2, U13 AMS1117-3.3, U14 USB2514B_Bi, Y2 24MHz, Y3 40MHz, Y4 40MHz, Y5 40MHz

Commit message: routing...
Parts:
- removed SW6, SW7, SW8: SW_Push, Button_Switch_SMD:SW_Tactile_SPST_NO_Straight_CK_PTS636Sx25SMTRLFS, symbol Switch:SW_Push
- added TP1, TP2, TP3: TestPoint, TestPoint:TestPoint_Pad_D1.5mm, symbol Connector:TestPoint
Connections:
- net at C30.1, R23.2, U10.4 (CHIP_PU/RESET): now also TP1.1
- net at C38.1, R37.2, U12.4 (CHIP_PU/RESET): now also TP3.1
- net at C34.1, R33.2, U11.4 (CHIP_PU/RESET): now also TP2.1

Commit message: routing...
Parts:
- AE3: footprint RF_Antenna:Texas_SWRA117D_2.4GHz_Left -> RF_Antenna:Texas_SWRA117D_2.4GHz_Right
Changed lines of the file:
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@@
 			)
 		)
-		(property "Footprint" "RF_Antenna:Texas_SWRA117D_2.4GHz_Left"
+		(property "Footprint" "RF_Antenna:Texas_SWRA117D_2.4GHz_Right"
 			(at 374.65 161.29 0)
 			(effects

Commit message: routing...
Parts:
- removed C37, C45, C46, C48, C49, C52, C53, C56, C57: 0.1uF, Capacitor_SMD:C_0603_1608Metric, symbol Device:C
- removed C47, C51, C55: 1uF, Capacitor_SMD:C_0603_1608Metric, symbol Device:C
- removed C50, C54: 10uF, Capacitor_SMD:C_0603_1608Metric, symbol Device:C
- removed FB5: FerriteBead, Inductor_SMD:L_0603_1608Metric, symbol Device:FerriteBead_Small
- added C12, C14, C16, C17, C18, C21, C23, C24, C5, C6, C7: 0.1uF, Capacitor_SMD:C_0603_1608Metric, symbol Device:C
- added C13, C15, C22: 10uF, Capacitor_SMD:C_0603_1608Metric, symbol Device:C
- added FB1, FB2: FerriteBead, Inductor_SMD:L_0603_1608Metric, symbol Device:FerriteBead_Small
- AE3: footprint RF_Antenna:Texas_SWRA117D_2.4GHz_Right -> RF_Antenna:Texas_SWRA117D_2.4GHz_Left
- C19: value 10uF -> 0.1uF; LCSC# C6119864 -> C5137636
Connections:
- net +3V3: now also C16.1, C17.1, C18.1, C23.1, C24.1, C6.1, FB1.2, FB2.2; no longer C19.2, C8.2, C9.1, U10.55 (VDDA), U10.56 (VDDA), U11.55 (VDDA), U11.56 (VDDA), U12.55 (VDDA), U12.56 (VDDA), U14.10 (VDDA33), U14.29 (VDDA33), U14.36 (VDDA33), U14.5 (VDDA33)
- net GND: now also C12.1, C13.1, C14.1, C15.1, C16.2, C17.2, C18.2, C21.1, C22.1, C23.2, C24.2, C5.1, C6.2, C7.1
- net VDD3P3: now also C19.2, U10.55 (VDDA), U10.56 (VDDA), U11.55 (VDDA), U11.56 (VDDA), U12.55 (VDDA), U12.56 (VDDA), C12.2, C13.2, C14.2, C15.2, C21.2, C22.2, C5.2, C7.2, FB1.1, FB2.1; no longer FB3.1
- new net vdda3v3: C8.2, C9.1, FB3.1, U14.10 (VDDA33), U14.29 (VDDA33), U14.36 (VDDA33), U14.5 (VDDA33)
- no-connect marks 79 -> 107
Other:
- note removed: "0.1 µF on VDD33 and 1 µF + 0.1 µF on the analog supply;"
