File: kicad/mdb-ai-bridge-esp32s3/mdb-ai-bridge-esp32s3.kicad_pcb (KiCad board)
At the start: 2 copper layers, 92 parts, among them J2 Conn_02x08_Top_Bottom, J7 USB_C_Receptacle_USB2.0_16P, SW3 SW_Push, SW4 SW_Push, SW5 SW_Push, SW6 SW_Push, SW7 SW_Push, SW8 SW_Push, SW9 SW_Push, U10 ESP32-S3FH4R2, U11 ESP32-S3FH4R2, U12 ESP32-S3FH4R2, U13 AMS1117-3.3, U14 USB2514B_Bi, Y2 Crystal_GND24, Y3 Crystal_GND24, Y4 Crystal_GND24, Y5 Crystal_GND24

Commit message: routing...
Parts:
- moved SW3 237.1 mm to (250.7, 93.0), turned to 180 degrees
- moved SW7 229.0 mm to (249.2, 83.8), turned to 180 degrees
- moved SW9 227.7 mm to (246.5, 102.5), turned to 180 degrees
- moved Y3 204.2 mm to (230.7, 103.9), turned to 180 degrees
- moved U10 184.9 mm to (230.1, 93.7), turned to 180 degrees
- moved D11 182.3 mm to (229.2, 85.0), turned to 180 degrees
- moved SW6 180.7 mm to (195.4, 96.9)
- moved SW5 180.1 mm to (195.6, 89.0)
- moved Y5 177.2 mm to (207.7, 85.0)
- moved D10 164.3 mm to (208.0, 101.7)
- moved U12 155.6 mm to (205.8, 92.8)
- moved Y2 149.4 mm to (177.1, 87.7)
- moved SW4 134.2 mm to (144.4, 89.2)
- moved SW8 128.6 mm to (144.1, 96.2)
- moved Y4 128.0 mm to (157.9, 82.7)
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Other:
- board outline added: 130.3 x 40 mm

Commit message: routing...
Parts:
- removed D8: D_Schottky, Diode_SMD:D_SOD-123
- removed J2: Conn_02x08_Top_Bottom, Connector_PinHeader_2.54mm:PinHeader_2x08_P2.54mm_Vertical
- added C3: 1uF, Capacitor_SMD:C_0603_1608Metric, F.Cu at (641.0, 244.4)
- added C4: 0.1uF, Capacitor_SMD:C_0603_1608Metric, F.Cu at (70.6, 137.0)
- added J3: Conn_02x08_Top_Bottom, Connector_PinHeader_2.54mm:PinHeader_2x08_P2.54mm_Vertical, F.Cu at (63.7, 135.5)
- added R10: 10k, Resistor_SMD:R_0603_1608Metric, F.Cu at (635.5, 230.9)
- C2: value 0.1uF -> 1uF
- R2, R3: value 100k -> 10k
- R8, R9: value 10k -> 100k
- moved C10 643.5 mm to (642.6, 230.8), turned to 90 degrees
- moved C20 642.9 mm to (638.7, 248.2), turned to 90 degrees
- moved C11 638.5 mm to (632.3, 248.3), turned to -90 degrees
- moved C1 637.3 mm to (630.3, 240.4), turned to 180 degrees
- moved C8 633.5 mm to (630.2, 231.6)
- moved C9 633.4 mm to (630.2, 233.6), turned to 180 degrees
- moved R11 632.2 mm to (640.9, 242.8), turned to 180 degrees
- moved R2 628.9 mm to (640.9, 230.8), turned to 90 degrees
- moved R42 628.8 mm to (637.8, 257.3), turned to 90 degrees
- moved R41 628.2 mm to (637.9, 252.8), turned to 90 degrees
- moved C41 627.6 mm to (625.0, 255.2), turned to 180 degrees
- moved C42 625.9 mm to (625.0, 252.7), turned to 180 degrees
- moved R4 625.5 mm to (635.0, 243.1)
- moved R3 624.6 mm to (637.2, 230.9), turned to 90 degrees
- moved R1 623.1 mm to (630.2, 242.0)
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Connections:
- C2 pad 1: +3V3 -> GND
- C2 pad 2: GND -> Net-(U14-CRFILT)
- C42 pad 2: /vin -> +5V
- J7 pad A4: Net-(D8-A) -> +5V
- J7 pad A9: Net-(D8-A) -> +5V
- J7 pad B4: Net-(D8-A) -> +5V
- J7 pad B9: Net-(D8-A) -> +5V
- R2 pad 1: GND -> Net-(U14-PRTPWR1/BC_EN1)
- R2 pad 2: Net-(U14-SCL/SMBCLK/CFG_SEL0) -> GND
- R3 pad 1: GND -> Net-(U14-PRTPWR2/BC_EN2)
- R3 pad 2: Net-(U14-SDA/SMBDATA/NON_REM1) -> GND
- R5 pad 1: +3V3 -> GND
- R7 pad 1: Net-(D8-A) -> +5V
- R8 pad 1: Net-(U14-USBDM_DN4/PRT_DIS_M4) -> GND
- R8 pad 2: +3V3 -> Net-(U14-SCL/SMBCLK/CFG_SEL0)
- R9 pad 1: Net-(U14-USBDP_DN4/PRT_DIS_P4) -> GND
- R9 pad 2: +3V3 -> Net-(U14-SDA/SMBDATA/NON_REM1)
- U11 pad 24: unconnected-(U11-GPIO18/ADC2_CH7-Pad24) -> /io18
- U13 pad 3: /vin -> +5V
- U14 pad 12: unconnected-(U14-PRTPWR1/BC_EN1-Pad12) -> Net-(U14-PRTPWR1/BC_EN1)
- U14 pad 13: unconnected-(U14-OCS_N1-Pad13) -> +3V3
- U14 pad 14: unconnected-(U14-CRFILT-Pad14) -> Net-(U14-CRFILT)
- U14 pad 16: unconnected-(U14-PRTPWR2/BC_EN2-Pad16) -> Net-(U14-PRTPWR2/BC_EN2)
- U14 pad 17: unconnected-(U14-OCS_N2-Pad17) -> +3V3
- U14 pad 18: unconnected-(U14-PRTPWR3/BC_EN3-Pad18) -> Net-(U14-PRTPWR3/BC_EN3)
- U14 pad 19: unconnected-(U14-OCS_N3-Pad19) -> +3V3
- U14 pad 21: unconnected-(U14-OCS_N4-Pad21) -> +3V3
- U14 pad 34: unconnected-(U14-PLLFILT-Pad34) -> Net-(U14-PLLFILT)
- U14 pad 8: Net-(U14-USBDM_DN4/PRT_DIS_M4) -> unconnected-(U14-USBDM_DN4/PRT_DIS_M4-Pad8)
- U14 pad 9: Net-(U14-USBDP_DN4/PRT_DIS_P4) -> unconnected-(U14-USBDP_DN4/PRT_DIS_P4-Pad9)

Commit message: routing...
Parts:
- moved C10 417.3 mm to (252.2, 83.5)
- moved C20 417.3 mm to (248.3, 100.8)
- moved C3 417.3 mm to (250.6, 97.0)
- moved C9 417.3 mm to (239.8, 86.2)
- moved R1 417.3 mm to (239.8, 94.6)
- moved R5 417.3 mm to (239.9, 91.4)
- moved R8 417.3 mm to (239.9, 89.6)
- moved U14 417.3 mm to (247.7, 90.2)
- moved Y2 417.3 mm to (245.3, 100.8)
- moved C1 417.3 mm to (239.9, 93.0)
- moved C11 417.3 mm to (241.9, 100.9)
- moved C2 417.3 mm to (248.6, 83.5)
- moved C8 417.3 mm to (239.8, 84.2)
- moved J7 417.3 mm to (254.3, 108.6)
- moved R10 417.3 mm to (245.1, 83.5)
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