File: kicad/mdb-bridge-esp32s3/mdb-bridge-esp32s3.kicad_sch (KiCad schematic)
At the start: 53 parts, among them J1 MDB_Connector, J2 USB_C_Receptacle_USB2.0_16P, J4 Conn_Coaxial, J8 Conn_01x04_Pin, J9 MDB_Connector, Q8 MMBT3904, SW1 SW_Push, U1 TLP785, U3 ESP32-S3FH4R2, U4 TLP785, U5 LM2594HVM-3.3, U7 MT3608, Y1 Crystal_GND24

Commit message: refacting
Parts:
- C22: value 22pF -> 22uF; LCSC# C105620 -> (none)
- L5: value 4.7uF -> 4.7uH
Changed lines of the file:
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@@
 			)
 		)
-		(property "Value" "22pF"
+		(property "Value" "22uF"
 			(at 368.3 193.0399 0)
 			(effects
@@
 			)
 		)
-		(property "LCSC#" "C105620"
+		(property "LCSC#" ""
 			(at 364.49 191.77 90)
 			(effects
@@
 			)
 		)
-		(property "Value" "4.7uF"
+		(property "Value" "4.7uH"
 			(at 332.74 170.18 90)
 			(effects
