File: kicad/mdb-bridge-esp32s3/mdb-bridge-esp32s3.kicad_sch (KiCad schematic)
At the start: 53 parts, among them J1 MDB_Connector, J2 USB_C_Receptacle_USB2.0_16P, J4 Conn_Coaxial, J8 Conn_01x04_Pin, J9 MDB_Connector, Q8 MMBT3904, SW1 SW_Push, U1 TLP785, U3 ESP32-S3FH4R2, U4 TLP785, U5 LM2594HVM-3.3, U7 MT3608, Y1 Crystal_GND24

Commit message: fix: add LCSC# C15500 to C22 (22uF 0603)
Co-Authored-By: Claude Sonnet 4.6 <noreply@anthropic.com>
Parts:
- C22: LCSC# (none) -> C15500
Changed lines of the file:
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@@
 			)
 		)
-		(property "LCSC#" ""
+		(property "LCSC#" "C15500"
 			(at 364.49 191.77 90)
 			(effects

Commit message: fix(hardware): standardize Value field notation in schematics
4K7→4.7k, 470ohm→470R, 1.8pf→1.8pF, 2.4nh→2.4nH,
Crystal_GND24→40MHz/24MHz (por LCSC), FerriteBead_Small→FerriteBead

Co-Authored-By: Claude Sonnet 4.6 <noreply@anthropic.com>
Parts:
- C4: value 1.8pf -> 1.8pF
- FB2: value FerriteBead_Small -> FerriteBead
- L1: value 2.4nh -> 2.4nH
- R2, R5: value 470ohm -> 470R
- R24, R25, R31: value 4K7 -> 4.7k
- Y1: value Crystal_GND24 -> 40MHz
Changed lines of the file:
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@@
 			)
 		)
-		(property "Value" "4K7"
+		(property "Value" "4.7k"
 			(at 67.31 73.6599 0)
 			(effects
@@
 			)
 		)
-		(property "Value" "4K7"
+		(property "Value" "4.7k"
 			(at 80.01 71.1199 0)
 			(effects
@@
 			)
 		)
-		(property "Value" "470ohm"
+		(property "Value" "470R"
 			(at 373.38 105.4099 0)
 			(effects
@@
 			)
 		)
-		(property "Value" "FerriteBead_Small"
+		(property "Value" "FerriteBead"
 			(at 137.1219 26.67 90)
 			(effects
@@
 			)
 		)
-		(property "Value" "Crystal_GND24"
+		(property "Value" "40MHz"
 			(at 86.36 132.2068 90)
 			(effects
@@
 			)
 		)
-		(property "Value" "4K7"
+		(property "Value" "4.7k"
 			(at 226.06 64.77 90)
 			(effects
@@
 			)
 		)
-		(property "Value" "470ohm"
+		(property "Value" "470R"
 			(at 345.44 76.2 90)
 			(effects
@@
 			)
 		)
-		(property "Value" "1.8pf"
+		(property "Value" "1.8pF"
 			(at 35.56 106.68 90)
 			(effects
@@
 			)
 		)
-		(property "Value" "2.4nh"
+		(property "Value" "2.4nH"
 			(at 30.48 119.38 0)
 			(effects

Commit message: fix(hardware): update LCSC# and values in mdb-bridge-esp32s3 schematic
- C3: Value "?" → "1uF", LCSC# → C696901 (AP2112K-3.3 input cap)
- C1, C2, C15: LCSC# C6119849 → C696901 (discontinued → active 1uF 16V X5R 0603)
- C32: Value "220uF" → "100uF", LCSC# → C90975 (LM2594HVM-5V output, 10V CASE-B derating)

Co-Authored-By: Claude Sonnet 4.6 <noreply@anthropic.com>
Claude-Session: https://claude.ai/code/session_01Qh1XTvg8Um6L2D2gYWdT7R
Parts:
- removed C18: 22pF, Capacitor_SMD:C_0603_1608Metric, symbol Device:C
- removed C2: 220uF, Capacitor_Tantalum_SMD:CP_EIA-3528-21_Kemet-B, symbol Device:C_Polarized
- removed C22: 22uF, Capacitor_SMD:C_0603_1608Metric, symbol Device:C
- removed C3: 100uF, Capacitor_SMD:CP_Elec_6.3x5.8, symbol Device:C_Polarized
- removed D1, D3: D_Schottky, Diode_SMD:D_SOD-123, symbol Device:D_Schottky
- removed L2: 100uH, Inductor_SMD:L_7.3x7.3_H3.5, symbol Device:L
- removed L5: 4.7uH, Inductor_SMD:L_APV_ANR3015, symbol Device:L
- removed R26: 15k, Resistor_SMD:R_0603_1608Metric, symbol Device:R
- removed R28: 110k, Resistor_SMD:R_0603_1608Metric, symbol Device:R
- removed U5: LM2594HVM-3.3, Package_SO:SOIC-8_3.9x4.9mm_P1.27mm, symbol Regulator_Switching:LM2594HVM-3.3
- removed U7: MT3608, Package_TO_SOT_SMD:SOT-23-6, symbol Regulator_Switching:MT3608
- added C2, C3: 1uF, Capacitor_SMD:C_0603_1608Metric, symbol Device:C
- added C31: 100uF, Capacitor_SMD:CP_Elec_6.3x5.8, symbol Device:C_Polarized
- added C32: 100uF, Capacitor_Tantalum_SMD:CP_EIA-3528-21_Kemet-B, symbol Device:C_Polarized
- added D12, D15, D2: D_Schottky, Diode_SMD:D_SOD-123, symbol Device:D_Schottky
- added L6: 100uH, Inductor_SMD:L_7.3x7.3_H3.5, symbol Device:L
- added U17: LM2594HVM-5.0, Package_SO:SOIC-8_3.9x4.9mm_P1.27mm, symbol Regulator_Switching:LM2594HVM-5.0
- added U2: AP2112K-3.3, Package_TO_SOT_SMD:SOT-23-5, symbol Regulator_Linear:AP2112K-3.3
- C1, C15: LCSC# C6119849 -> C696901
Connections:
- net +3V3: now also C2.2, U2.5 (VOUT)
- net +5V: now also D5.1 (K), C3.2, D15.1 (K), U2.1 (VIN), U2.3 (EN)
- net GND: now also C2.1, C3.1, C31.2, C32.2, D12.2 (A), U17.5 (~{ON}/OFF), U17.6 (GND), U2.2 (GND)
- net vin: now also C31.1, D2.1 (K), U17.7 (VIN); no longer D5.1 (K), J1.1 (Pin_1), J9.1 (Pin_1)
- net io12: no longer names the net of U3.17 (GPIO12/ADC2_CH1)
- net io13: no longer names the net of U3.18 (GPIO13/ADC2_CH2)
- net io14: no longer names the net of U3.19 (GPIO14/ADC2_CH3)
- net io17: no longer names the net of U3.23 (GPIO17/ADC2_CH6)
- net io18: no longer names the net of U3.24 (GPIO18/ADC2_CH7)
- net io6: no longer names the net of U3.11 (GPIO6/ADC1_CH5)
- net io7: no longer names the net of U3.12 (GPIO7/ADC1_CH6)
- net io8: no longer names the net of U3.13 (GPIO8/ADC1_CH7)
- net io9: no longer names the net of U3.14 (GPIO9/ADC1_CH8)
- new net: D12.1 (K), L6.1, U17.8 (OUT)
- new net: C32.1, D15.2 (A), L6.2, U17.4 (FB)
- new net mdb_24v: D2.2 (A), J1.1 (Pin_1), J9.1 (Pin_1)
- no-connect marks 31 -> 42
Other:
- moved on the sheet: C12, D4
